File: timer/a02_3.kicad_sch (KiCad schematic)
At the start: 23 parts, among them U2024 74HC27, U2025 74HC02, U2026 74HC02, U2027 74HC02, U2028 74HC27, U2029 74HC02, U2030 74HC02, U2031 74HC27, U2032 74HC02, U2033 74HC02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

Commit message: Added Init values
Added individual Init Values for Components. TImer Module Updated with init values
Parts:
- U2024: Init_A (none) -> 1; Init_B (none) -> 0; Init_C (none) -> 0; Init_D (none) -> 0; Initial 1 -> (none)
- U2024: Init_A (none) -> 1; Init_B (none) -> 0; Init_C (none) -> 0; Init_D (none) -> 0
- U2025: Init_A (none) -> 0; Init_B (none) -> 0; Init_C (none) -> 0; Init_D (none) -> 1
- U2025: Init_A (none) -> 0; Init_B (none) -> 0; Init_C (none) -> 0; Init_D (none) -> 1; Initial 1 -> (none)
- U2026, U2030, U2035: Init_A (none) -> 0; Init_B (none) -> 0; Init_C (none) -> 1; Init_D (none) -> 0
- U2026, U2030, U2035: Init_A (none) -> 0; Init_B (none) -> 0; Init_C (none) -> 1; Init_D (none) -> 0; Initial 1 -> (none)
- U2027, U2032, U2036: Init_A (none) -> 0; Init_B (none) -> 1; Init_C (none) -> 0; Init_D (none) -> 0
- U2027, U2032, U2036: Init_A (none) -> 0; Init_B (none) -> 1; Init_C (none) -> 0; Init_D (none) -> 0; Initial 1 -> (none)
- U2028, U2031, U2034, U2037, U2041, U2044: Init_A (none) -> 0; Init_B (none) -> 0; Init_C (none) -> 0; Init_D (none) -> 0
- U2029, U2033: Init_A (none) -> 1; Init_B (none) -> 0; Init_C (none) -> 0; Init_D (none) -> 1; Initial 1 -> (none)
- U2029, U2033: Init_A (none) -> 1; Init_B (none) -> 0; Init_C (none) -> 0; Init_D (none) -> 1
- U2039, U2040, U2042: Init_A (none) -> 0; Init_B (none) -> 0; Init_C (none) -> 0; Init_D (none) -> 0; Init_E (none) -> 0; Init_F (none) -> 0
