File: timer/clock_divider.kicad_sch (KiCad schematic)
At the start: 2 parts, among them U2101 74HC02, U2102 74HC27

Commit message: Added Init values
Added individual Init Values for Components. TImer Module Updated with init values
Parts:
- U2101, U2102: Init_A (none) -> 0; Init_B (none) -> 1; Init_C (none) -> 0; Init_D (none) -> 0
- U2101, U2102: Init_A (none) -> 0; Init_B (none) -> 1; Init_C (none) -> 0; Init_D (none) -> 0; Initial 1 -> (none)
Changed lines of the file:
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@@
       (effects (font (size 1.524 1.524)))
+    )
+    (property "Init_A" "0" (id 4) (at 59.69 88.9 0)
+      (effects (font (size 1.27 1.27)) hide)
+    )
+    (property "Init_B" "1" (id 5) (at 60.96 88.9 0)
+      (effects (font (size 1.27 1.27)) hide)
+    )
+    (property "Init_C" "0" (id 6) (at 62.23 88.9 0)
+      (effects (font (size 1.27 1.27)) hide)
+    )
+    (property "Init_D" "0" (id 7) (at 63.5 88.9 0)
+      (effects (font (size 1.27 1.27)) hide)
     )
     (pin "1")
@@
       (effects (font (size 1.524 1.524)))
     )
-    (property "Initial" "1" (id 4) (at 68.58 87.63 0)
-      (effects (font (size 1.524 1.524) italic))
+    (property "Init_A" "0" (id 4) (at 59.69 88.9 0)
+      (effects (font (size 1.27 1.27)) hide)
+    )
+    (property "Init_B" "1" (id 5) (at 60.96 90.17 0))
+    (property "Init_C" "0" (id 6) (at 62.23 88.9 0)
+      (effects (font (size 1.27 1.27)) hide)
+    )
+    (property "Init_D" "0" (id 7) (at 63.5 88.9 0)
+      (effects (font (size 1.27 1.27)) hide)
     )
     (pin "1")
@@
       (effects (font (size 1.524 1.524)))
     )
+    (property "Init_A" "0" (id 5) (at 97.79 35.56 0)
+      (effects (font (size 1.27 1.27)) hide)
+    )
+    (property "Init_B" "1" (id 6) (at 100.33 72.39 0)
+      (effects (font (size 1.27 1.27)) hide)
+    )
+    (property "Init_C" "0" (id 7) (at 97.79 73.66 0)
+      (effects (font (size 1.27 1.27)) hide)
+    )
+    (property "Init_D" "0" (id 8) (at 97.79 71.12 0)
+      (effects (font (size 1.27 1.27)) hide)
+    )
     (pin "1")
     (pin "2")
@@
       (effects (font (size 1.524 1.524)))
     )
+    (property "Init_A" "0" (id 5) (at 97.79 142.24 0)
+      (effects (font (size 1.27 1.27)) hide)
+    )
+    (property "Init_B" "1" (id 6) (at 97.79 71.12 0)
+      (effects (font (size 1.27 1.27)) hide)
+    )
+    (property "Init_C" "0" (id 7) (at 97.79 71.12 0)
+      (effects (font (size 1.27 1.27)) hide)
+    )
+    (property "Init_D" "0" (id 8) (at 97.79 71.12 0)
+      (effects (font (size 1.27 1.27)) hide)
+    )
     (pin "1")
     (pin "2")
@@
       (effects (font (size 1.524 1.524)))
     )
-    (property "Initial" "1" (id 4) (at 102.87 69.85 0)
-      (effects (font (size 1.524 1.524) italic))
+    (property "Init_A" "0" (id 5) (at 100.33 72.39 0)
+      (effects (font (size 1.27 1.27)) hide)
+    )
+    (property "Init_B" "1" (id 6) (at 95.25 72.39 0))
+    (property "Init_C" "0" (id 7) (at 99.06 72.39 0)
+      (effects (font (size 1.27 1.27)) hide)
+    )
+    (property "Init_D" "0" (id 8) (at 96.52 73.66 0)
+      (effects (font (size 1.27 1.27)) hide)
     )
     (pin "1")
@@
       (effects (font (size 1.524 1.524)))
     )
-    (pin "1")
+    (property "Init_A" "0" (id 5) (at 97.79 106.68 0)
+      (effects (font (size 1.27 1.27)) hide)
+    )
+    (property "Init_B" "1" (id 6) (at 97.79 72.39 0)
+      (effects (font (size 1.27 1.27)) hide)
+    )
+    (property "Init_C" "0" (id 7) (at 97.79 71.12 0)
+      (effects (font (size 1.27 1.27)) hide)
+    )
+    (property "Init_D" "0" (id 8) (at 97.79 71.12 0)
+      (effects (font (size 1.27 1.27)) hide)
+    )
+    (pin "1")
