File: timer/timer.kicad_sch (KiCad schematic)
At the start: 49 parts, among them P1 DIN_41612_128P, U2024 74HC27, U2025 74HC02, U2026 74HC02, U2027 74HC02, U2028 74HC27, U2029 74HC02, U2030 74HC02, U2031 74HC27, U2032 74HC02, U2033 74HC02, U2034 74HC27, U2035 74HC02, U2036 74HC02, U2037 74HC27, U2038 74LVC07, U2039 74HC04, U2040 74HC04, U2041 74HC27, U2042 74HC04, U2043 74HC4002, U2044 74HC02, U2046 74LVC06, U2047 74LVC06, U2101 74HC02, U2102 74HC27, U2103 74HC04, U2104 74HC02, U2105 74HC04, U2106 74HC02, U2107 74HC27, U2108 74HC04, U2109 74HC02, U2110 74HC04, U2111 74HC27, U2112 74HC02, U2113 74HC02, U2114 74HC02, U2115 74HC02, U2116 74HC02, U2117 74HC02, U2118 74HC27, U2119 74HC27, U2120 74LVC07, U2121 74HC04, U2122 74HC02, U2123 74HC02, U2145 74HC04, U2148 74LVC06

Commit message: Added Init values
Added individual Init Values for Components. TImer Module Updated with init values
Parts:
- U2024: Init_A (none) -> 1; Init_B (none) -> 0; Init_C (none) -> 0; Init_D (none) -> 0
- U2025: Init_A (none) -> 0; Init_B (none) -> 0; Init_C (none) -> 0; Init_D (none) -> 1
- U2026, U2030, U2035: Init_A (none) -> 0; Init_B (none) -> 0; Init_C (none) -> 1; Init_D (none) -> 0
- U2027, U2032, U2036, U2101, U2102, U2112, U2113, U2114, U2115: Init_A (none) -> 0; Init_B (none) -> 1; Init_C (none) -> 0; Init_D (none) -> 0
- U2028, U2031, U2034, U2037, U2041, U2044, U2104, U2106, U2107, U2111, U2117, U2118, U2119, U2122: Init_A (none) -> 0; Init_B (none) -> 0; Init_C (none) -> 0; Init_D (none) -> 0
- U2029, U2033: Init_A (none) -> 1; Init_B (none) -> 0; Init_C (none) -> 0; Init_D (none) -> 1
- U2039, U2040, U2042, U2103, U2108, U2110, U2121, U2145: Init_A (none) -> 0; Init_B (none) -> 0; Init_C (none) -> 0; Init_D (none) -> 0; Init_E (none) -> 0; Init_F (none) -> 0
- U2105: Init_A (none) -> 0; Init_B (none) -> 0; Init_C (none) -> 0; Init_D (none) -> 0; Init_E (none) -> 1; Init_F (none) -> 0
- U2109, U2123: Init_A (none) -> 0; Init_B (none) -> 1; Init_C (none) -> 0; Init_D (none) -> 1
- U2116: Init_A (none) -> 0; Init_B (none) -> 1; Init_C (none) -> 1; Init_D (none) -> 0
Connections:
- no-connect marks 18 -> 19
