File: four_bit_generic/two_bit_columns.kicad_sch (KiCad schematic)
At the start: 49 parts

Commit message: Generic  4 Bit Adder schematic + pcb
PCB and schematic updates
Parts:
- added A8_R10: 5k, agc_footprints:R_0603_1608Metric, symbol Device:R
- added unit 3 of UA8_11
- added unit 2 of UA8_11
- added unit 3 of UA8_15
- added unit 4 of UA8_16
- added unit 2 of UA8_16
- added unit 5 of UA8_16
- added unit 2 of UA8_2
- added unit 6 of UA8_2
- added unit 5 of UA8_2
- added unit 5 of UA8_22
- added unit 3 of UA8_22
- added unit 1 of UA8_22
- added unit 4 of UA8_25
- added unit 1 of UA8_27
- added unit 3 of UA8_31
- added unit 2 of UA8_31
- added unit 3 of UA8_35
- added unit 5 of UA8_36
- added unit 4 of UA8_36
- added unit 1 of UA8_36
- added unit 4 of UA8_5
- added unit 6 of UA8_7
Connections:
- net +4VSW: now also A8_R10.1
- net GND: now also UA8_11.10, UA8_11.11, UA8_11.3, UA8_11.4, UA8_11.5, UA8_11.9, UA8_15.8, UA8_15.9, UA8_16.11, UA8_16.3, UA8_16.9, UA8_2.13, UA8_2.3, UA8_22.11, UA8_27.1, UA8_31.3, UA8_31.4, UA8_31.5, UA8_35.8, UA8_35.9, UA8_36.1, UA8_36.9, UA8_5.11, UA8_5.12, UA8_7.13
- net X2/: now also UA8_13.3; no longer UA8_13.2
- net Y2/: now also UA8_13.2; no longer UA8_13.3
- net _MWL1: now also UA8_22.4; no longer UA8_22.6
- net _WL1: now also UA8_22.3; no longer UA8_22.5
- new net BUF_PU_SPARE_1_IN: UA8_22.1
- new net BUF_PU_SPARE_1_OUT: A8_R10.2, UA8_22.2
- new net BUF_SPARE_1_IN: UA8_22.5
- new net BUF_SPARE_1_OUT: UA8_22.6
- new net BUF_SPARE_2_IN: UA8_2.11
- new net BUF_SPARE_2_OUT: UA8_2.10
- new net BUF_SPARE_3_IN: UA8_36.11
- new net BUF_SPARE_3_OUT: UA8_36.10
- new net NOR_2_SPARE_1_IN_1: UA8_25.11
- new net NOR_2_SPARE_1_IN_2: UA8_25.12
- new net NOR_2_SPARE_1_OUT: UA8_25.13
- new net NOR_3_SPARE_1_IN_1: UA8_31.9
- new net NOR_3_SPARE_1_IN_2: UA8_31.10
- new net NOR_3_SPARE_1_IN_3: UA8_31.11
- new net NOR_3_SPARE_1_OUT: UA8_31.8
- no-connect marks 0 -> 16
Other:
- note added: "Connected Spare Gates"
- note added: "Unused Gates"
