File: four_bit_generic/two_bit_columns_B.kicad_sch (KiCad schematic)
At the start: 49 parts

Commit message: Generic  4 Bit Adder schematic + pcb
PCB and schematic updates
Parts:
- added A8_R50: 5k, agc_footprints:R_0603_1608Metric, symbol Device:R
- added unit 5 of UA8_42
- added unit 6 of UA8_42
- added unit 2 of UA8_42
- added unit 3 of UA8_45
- added unit 3 of UA8_47
- added unit 2 of UA8_51
- added unit 1 of UA8_51
- added unit 4 of UA8_55
- added unit 5 of UA8_56
- added unit 2 of UA8_56
- added unit 6 of UA8_56
- added unit 3 of UA8_62
- added unit 6 of UA8_62
- added unit 1 of UA8_62
- added unit 3 of UA8_65
- added unit 3 of UA8_67
- added unit 2 of UA8_71
- added unit 3 of UA8_71
- added unit 3 of UA8_75
- added unit 6 of UA8_76
- added unit 3 of UA8_76
- added unit 2 of UA8_76
Connections:
- net +4VSW: now also A8_R50.1
- net GND: now also UA8_54.5, UA8_42.11, UA8_42.3, UA8_45.8, UA8_45.9, UA8_47.5, UA8_51.1, UA8_51.13, UA8_51.2, UA8_51.3, UA8_51.4, UA8_51.5, UA8_55.11, UA8_55.12, UA8_56.11, UA8_56.13, UA8_56.3, UA8_62.13, UA8_67.5, UA8_71.3, UA8_71.4, UA8_71.5, UA8_75.8, UA8_75.9, UA8_76.3, UA8_76.5; no longer UA8_54.1
- net RLG/: now also UA8_54.1; no longer UA8_54.10
- net X2/: now also UA8_53.2; no longer UA8_53.3
- net Y2/: now also UA8_53.3; no longer UA8_53.2
- net _CLG: now also UA8_54.3; no longer UA8_54.13
- net _L2/: now also UA8_54.2, UA8_54.4; no longer UA8_54.2, UA8_54.9
- net _LINH_2: now also UA8_54.13; no longer UA8_54.11
- net _MWL1: now also UA8_62.4; no longer UA8_62.2
- net _RL_OUT_2: now also UA8_54.12; no longer UA8_54.8
- net _RUG_1: now also UA8_71.1; no longer UA8_71.11
- net _SUMA1: now also UA8_71.2; no longer UA8_71.10
- net _SUMB1: now also UA8_71.13; no longer UA8_71.9
- net _WL1: now also UA8_62.3; no longer UA8_62.1
- net at UA8_77.9: now also UA8_71.12; no longer UA8_71.8
- net at UA8_55.1: now also UA8_54.9; no longer UA8_54.5
- net at UA8_55.10: now also UA8_54.10; no longer UA8_54.4
- net at UA8_56.1: now also UA8_54.8; no longer UA8_54.6
- new net: UA8_54.11, UA8_54.6
- new net BUF_PU_SPARE_2_IN: UA8_62.5
- new net BUF_PU_SPARE_2_OUT: A8_R50.2, UA8_62.6
- new net BUF_SPARE_4_IN: UA8_62.1
- new net BUF_SPARE_4_OUT: UA8_62.2
- new net BUF_SPARE_5_IN: UA8_42.13
- new net BUF_SPARE_5_OUT: UA8_42.12
- new net BUF_SPARE_6_IN: UA8_76.13
- new net BUF_SPARE_6_OUT: UA8_76.12
- new net NOR_2_SPARE_2_IN_1: UA8_65.8
- new net NOR_2_SPARE_2_IN_2: UA8_65.9
- new net NOR_2_SPARE_2_OUT: UA8_65.10
- new net NOR_3_SPARE_2_IN_1: UA8_71.9
- new net NOR_3_SPARE_2_IN_2: UA8_71.10
- new net NOR_3_SPARE_2_IN_3: UA8_71.11
- new net NOR_3_SPARE_2_OUT: UA8_71.8
- no-connect marks 0 -> 16
Other:
- note added: "Connected Spare Gates"
- note added: "Unused Gates"
