File: four_bit_generic/two_bit_colums_side2.kicad_sch (KiCad schematic)
At the start: 86 parts

Commit message: Generic  4 Bit Adder schematic + pcb
PCB and schematic updates
Parts:
- UA8_71: Initial 1 -> (none)
Other:
- sheet Generic_two_bit_columns1 ports: added BUF_PU_SPARE_2_IN, BUF_PU_SPARE_2_OUT, BUF_SPARE_4_IN, BUF_SPARE_4_OUT, BUF_SPARE_5_IN, BUF_SPARE_5_OUT, BUF_SPARE_6_IN, BUF_SPARE_6_OUT, NOR_2_SPARE_2_IN_1, NOR_2_SPARE_2_IN_2, NOR_2_SPARE_2_OUT, NOR_3_SPARE_2_IN_1, NOR_3_SPARE_2_IN_2, NOR_3_SPARE_2_IN_3, NOR_3_SPARE_2_OUT, _WLM_2/; removed _WLM_2/
- sheet two_bit_columns_side2_con ports: added BUF_PU_SPARE_2_IN, BUF_PU_SPARE_2_OUT, BUF_SPARE_4_IN, BUF_SPARE_4_OUT, BUF_SPARE_5_IN, BUF_SPARE_5_OUT, BUF_SPARE_6_IN, BUF_SPARE_6_OUT, NOR_2_SPARE_2_IN_1, NOR_2_SPARE_2_IN_2, NOR_2_SPARE_2_OUT, NOR_3_SPARE_2_IN_1, NOR_3_SPARE_2_IN_2, NOR_3_SPARE_2_IN_3, NOR_3_SPARE_2_OUT; removed none
- moved on the sheet: C47, C48, C49, C50, C51, C52, C53, C54, C55, C56, C57, C58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
